File: rf2mqtt/rf2mqtt.kicad_sch (KiCad schematic)
At the start: 21 parts, among them J1 Antenna Wire, Q1 TN0106N3-G, SW1 config, U1 Pico

Commit message: Use hardware timers for LED blink to work around asyncio limitations and allow a nice long sleep cycle for the main loop.
Parts:
- SW1: footprint Button_Switch_THT:SW_PUSH_1P1T_6x3.5mm_H4.3_APEM_MJTP1243 -> Button_Switch_THT:SW_PUSH_6mm_H13mm
Changed lines of the file:
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@@
 			)
 		)
-		(property "Footprint" "Button_Switch_THT:SW_PUSH_1P1T_6x3.5mm_H4.3_APEM_MJTP1243"
+		(property "Footprint" "Button_Switch_THT:SW_PUSH_6mm_H13mm"
 			(at 160.02 140.97 0)
 			(effects
